File: Hardware/RoboHand/robohand.brd (EAGLE design)
At the start: 88.9 x 63.5 mm, 25 parts, among them IC1 LM1117MPX-3.3, IC2 STM32F10XCXT6, U1 LSM9DS1

Commit message: reainstall
Parts:
- added R4, R5, R6, R7, R8: EVUF3A, pot:EVUF
- added U2: HC_05, hc-05:BLUETOOTH_SMD
- JP1, JP2: value (none) -> 0R-JUMPA; device pinhead:1X03/90 -> jump-0r-smd:A0R-JMP
- moved R1 123.8 mm to (76.5, 50.3)
- moved R2 120.3 mm to (68.1, 47.5), turned to 90 degrees
- moved C14 118.2 mm to (76.2, 45.7)
- moved U1 115.1 mm to (71.9, 51.1)
- moved C11 110.4 mm to (81.0, 46.5)
- moved JP2 110.1 mm to (63.2, 46.2)
- moved C13 108.3 mm to (71.6, 55.9), turned to 90 degrees
- moved C12 104.4 mm to (77.2, 57.7)
- moved C3 102.6 mm to (50.8, 49.5), turned to 180 degrees
- moved C2 100.7 mm to (58.2, 65.0)
- moved C15 100.2 mm to (68.1, 55.9), turned to 90 degrees
- moved JP1 97.7 mm to (59.9, 46.2)
- moved C1 90.6 mm to (57.1, 54.6)
- moved IC1 87.9 mm to (50.8, 58.4)
- moved C4 87.9 mm to (38.4, 64.5), turned to 315 degrees
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Connections:
- new net POT1: R4.2
- new net POT2: R5.2
- new net POT3: R6.2
- new net POT4: R7.2
- new net POT5: R8.2
- net +3V3: now also R4.1, R5.1, R6.1, R7.1, R8.1
- net GND: now also R4.3, R5.3, R6.3, R7.3, R8.3
Routing:
- net +3V3: track 0.00 -> 119.4 mm, vias 0 -> 2
- net GND: track 0.00 -> 65.5 mm
- net VCC: track 0.00 -> 17.4 mm
- net OSC_IN: track 0.00 -> 13.6 mm
- net OSC_OUT: track 0.00 -> 10.4 mm
