File: Hardware/RoboHand/robohand.sch (EAGLE design)
At the start: 25 parts, among them IC1 LM1117MPX-3.3, IC2 STM32F10XCXT6, U1 LSM9DS1

Commit message: reainstall
Parts:
- added R4, R5, R6, R7, R8: EVUF3A, pot:EVUF3A
- added U2: HC_05, hc-05:HC_05
- JP1, JP2: value (none) -> 0R-JUMPA; device pinhead:PINHD-1X3/90 -> jump-0r-smd:0R-JUMPA
Connections:
- new net POT1: R4.S
- new net POT2: R5.S
- new net POT3: R6.S
- new net POT4: R7.S
- new net POT5: R8.S
- net +3V3: now also JP1-0R.1, JP2-0R.1, R4.A, R5.A, R6.A, R7.A, R8.A; no longer JP1.1, JP2.1
- net GND: now also JP1-0R.3, JP2-0R.3, R4.E, R5.E, R6.E, R7.E, R8.E; no longer JP1.3, JP2.3
- net SDO_A/G: now also JP1-0R.2; no longer JP1.2
- net SDO_M: now also JP2-0R.2; no longer JP2.2
